File: hardware/bottom_board/bottom_board.kicad_pcb (KiCad board)
At the start: 2 copper layers, 27.2 x 27.2 mm, 25 parts, among them IC1 74HC595, IC2 74HC595, J1 Conn_01x06_Socket, J2 Conn_01x06_Socket, Q1 Q_PNP_BCE, Q2 Q_PNP_BCE, Q3 Q_PNP_BCE, Q4 Q_PNP_BCE, Q5 Q_PNP_BCE, Q6 Q_PNP_BCE, SW1 SW_SPDT, U1 ATtiny1616-M, U2 LIS3DH

Commit message: Recent changes
Parts:
- added TP1: TestPoint, TestPoint:TestPoint_Pad_D1.0mm, F.Cu at (108.6, 78.8)
- added TP2: TestPoint, TestPoint:TestPoint_Pad_D1.0mm, F.Cu at (108.6, 74.5)
- added TP3: TestPoint, TestPoint:TestPoint_Pad_D1.0mm, F.Cu at (108.6, 76.7)
- BT1: footprint Battery:BatteryHolder_MPD_BC2003_1x2032 -> Battery Holder CR2032-P28-K Compatible with CR2032 Horizontal SMT Reflow 24.2mm:BAT-SMD_MY-2032-12-Updated-4
- SW1: footprint SSSS811101:SW4_SSSS811101_ALPS -> SHOU HAN MINI MSK12CO2:SW-SMD_MSK12CO2
- U1: value ATtiny1616-M -> ATTINY1616-MNR; footprint Package_DFN_QFN:VQFN-20-1EP_3x3mm_P0.4mm_EP1.7x1.7mm -> MICROCHIP ATTINY1616-MNR:QFN-20_L3.0-W3.0-P0.40-BL-EP1.7
- moved C1 3.05 mm to (112.0, 76.2)
- moved SW1 3.02 mm to (113.8, 67.8), turned to 90 degrees
- moved R5 0.67 mm to (93.8, 71.7)
- moved R4 0.50 mm to (93.5, 80.2)
- moved U1 0.43 mm to (104.5, 76.4), turned to 90 degrees
- moved BT1 0.30 mm to (102.4, 76.4)
Connections:
- U1 pad 19: unconnected-(U1-~{RESET}/PA0-Pad19) -> Net-(U1-PA0/~{RESET}/UPDI)
- U1 pad 21: GND -> unconnected-(U1-EP-Pad21)
- U1 pad 5: /RCLK -> unconnected-(U1-PA4-Pad5)
- U1 pad 6: /SCLK -> /RCLK
- U1 pad 7: unconnected-(U1-PA6-Pad7) -> /SCLK
Routing:
- net Net-(U1-PA0/~{RESET}/UPDI): track 0.00 -> 13.8 mm, vias 0 -> 2
- net +3V0: track 123.7 -> 133.0 mm
- net /SCL: track 24.0 -> 28.2 mm
- net Net-(BT1-+): track 35.0 -> 38.2 mm
- net GND: track 82.6 -> 85.2 mm
- net /SCLK: track 57.0 -> 58.6 mm
- net /RCLK: track 39.4 -> 40.8 mm
- net Net-(Q5-B): track 2.74 -> 3.66 mm
- net /SDA: track 15.5 -> 16.2 mm
- net Net-(Q4-B): track 2.64 -> 3.35 mm
- net /TO_Q4: track 14.3 -> 13.7 mm
Other:
- board text added: "Dice by Faraz Aleboyeh, PCBA Sponsored by"
- board text removed: "Dice by Faraz Aleboyeh PCBA sponsored by"

Commit message: Recent changes
Parts:
- removed J2: Conn_01x06_Socket, Connector_PinSocket_1.27mm:PinSocket_1x06_P1.27mm_Vertical
- J1: value Conn_01x06_Socket -> Conn_01x12_Socket; footprint Connector_PinSocket_1.27mm:PinSocket_1x06_P1.27mm_Vertical -> Connector_PinSocket_1.27mm:PinSocket_1x12_P1.27mm_Vertical
- Q1, Q2, Q3, Q4, Q5, Q6: value Q_PNP_BCE -> Q_PNP_BEC
- R7, R8: value R -> 10k
- moved J1 8.68 mm to (95.2, 89.2)
- moved Q4 2.68 mm to (90.5, 78.0), turned to -90 degrees
- moved Q5 2.10 mm to (90.5, 74.3), turned to -90 degrees
- moved Q1 1.73 mm to (90.5, 89.5), turned to -90 degrees
- moved R5 1.58 mm to (93.8, 73.2)
- moved Q3 1.11 mm to (90.5, 82.0), turned to -90 degrees
- moved Q6 0.58 mm to (90.5, 70.5), turned to -90 degrees
- moved Q2 0.36 mm to (90.5, 85.8), turned to -90 degrees
Connections:
- J1 pad 1: /ROW1 -> /TO_Q1
- J1 pad 2: /ROW2 -> /TO_Q2
- J1 pad 3: /ROW3 -> /TO_Q3
- J1 pad 4: /ROW4 -> /TO_Q4
- J1 pad 5: /ROW5 -> /TO_Q5
- J1 pad 6: /ROW6 -> /TO_Q6
- Q1 pad 2: /TO_Q1 -> +3V0
- Q1 pad 3: +3V0 -> /TO_Q1
- Q2 pad 2: /TO_Q2 -> +3V0
- Q2 pad 3: +3V0 -> /TO_Q2
- Q3 pad 2: /TO_Q3 -> +3V0
- Q3 pad 3: +3V0 -> /TO_Q3
- Q4 pad 2: /TO_Q4 -> +3V0
- Q4 pad 3: +3V0 -> /TO_Q4
- Q5 pad 2: /TO_Q5 -> +3V0
- Q5 pad 3: +3V0 -> /TO_Q5
- Q6 pad 2: /TO_Q6 -> +3V0
- Q6 pad 3: +3V0 -> /TO_Q6
Routing:
- net +3V0: track 133.0 -> 140.2 mm, vias 6 -> 4
- net /SCLK: track 58.6 -> 53.3 mm, vias 6 -> 8
- net Net-(U1-PA0/~{RESET}/UPDI): track 13.8 -> 9.54 mm
- net /TO_Q5: track 22.3 -> 20.2 mm, vias 3 -> 1
- net GND: track 85.2 -> 83.3 mm
- net /COL5: track 5.97 -> 7.55 mm
- net Net-(Q5-B): track 3.66 -> 2.39 mm, vias 2 -> 0
- net Net-(Q2-B): track 2.80 -> 1.58 mm, vias 2 -> 0
- net Net-(Q6-B): track 2.73 -> 1.74 mm
- net /TO_Q1: track 5.93 -> 5.05 mm
- net Net-(Q3-B): track 2.80 -> 2.01 mm, vias 2 -> 0
- net /ROW1: track 10.2 -> 10.9 mm
- net /TO_Q4: track 13.7 -> 14.3 mm
- net Net-(Q4-B): track 3.35 -> 3.93 mm, vias 2 -> 0
- net /TO_Q6: track 26.6 -> 26.0 mm
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