File: hardware/bottom_board/bottom_board.kicad_sch (KiCad schematic)
At the start: 25 parts, among them IC1 74HC595, IC2 74HC595, J1 Conn_01x06_Socket, J2 Conn_01x06_Socket, Q1 Q_PNP_BCE, Q2 Q_PNP_BCE, Q3 Q_PNP_BCE, Q4 Q_PNP_BCE, Q5 Q_PNP_BCE, Q6 Q_PNP_BCE, SW1 SW_SPDT, U1 ATtiny1616-M, U2 LIS3DH

Commit message: Recent changes
Parts:
- removed U1: ATtiny1616-M, Package_DFN_QFN:VQFN-20-1EP_3x3mm_P0.4mm_EP1.7x1.7mm, symbol MCU_Microchip_ATtiny:ATtiny1616-M
- added TP1, TP2, TP3: TestPoint, TestPoint:TestPoint_Pad_D1.0mm, symbol Connector:TestPoint
- added U1: ATTINY1616-MNR, MICROCHIP ATTINY1616-MNR:QFN-20_L3.0-W3.0-P0.40-BL-EP1.7, symbol easyeda2kicad:ATTINY1616-MNR
- BT1: footprint Battery:BatteryHolder_MPD_BC2003_1x2032 -> Battery Holder CR2032-P28-K Compatible with CR2032 Horizontal SMT Reflow 24.2mm:BAT-SMD_MY-2032-12-Updated-4; LCSC Part (none) -> C6937139
- SW1: footprint SSSS811101:SW4_SSSS811101_ALPS -> SHOU HAN MINI MSK12CO2:SW-SMD_MSK12CO2; LCSC Part (none) -> C2681570
Connections:
- net +3V0: now also TP2.1, U1.4 (VDD)
- net DS: now also U1.2 (EXTCLK/PA3)
- net GND: now also TP3.1, U1.3 (GND)
- net INT: now also U1.15 (PC0)
- net RCLK: now also U1.6 (PA5)
- net SCL: now also U1.1 (PA2)
- net SCLK: now also U1.7 (PA6)
- net SDA: now also U1.20 (PA1)
- new net: TP1.1, U1.19 (PA0/~{RESET}/UPDI)
Other:
- moved on the sheet: BT1, C1, C2, C3, IC1, IC2, J1, J2, Q1, Q2, Q3, Q4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

Commit message: Recent changes
Parts:
- removed J1, J2: Conn_01x06_Socket, Connector_PinSocket_1.27mm:PinSocket_1x06_P1.27mm_Vertical, symbol Connector:Conn_01x06_Socket
- removed Q1, Q4: Q_PNP_BCE, Package_TO_SOT_SMD:SOT-523, symbol Transistor_BJT:Q_PNP_BCE
- added J1: Conn_01x12_Socket, Connector_PinSocket_1.27mm:PinSocket_1x12_P1.27mm_Vertical, symbol Connector:Conn_01x12_Socket
- added Q1, Q4: Q_PNP_BEC, Package_TO_SOT_SMD:SOT-523, symbol Transistor_BJT:Q_PNP_BEC
- Q2, Q3, Q5, Q6: value Q_PNP_BCE -> Q_PNP_BEC; symbol Transistor_BJT:Q_PNP_BCE -> Transistor_BJT:Q_PNP_BEC
- R7, R8: value R -> 10k
Connections:
- net +3V0: now also Q2.2 (E), Q3.2 (E), Q5.2 (E), Q6.2 (E), Q1.2 (E), Q4.2 (E); no longer Q2.3 (E), Q3.3 (E), Q5.3 (E), Q6.3 (E)
- net ROW1: now also J1.7 (Pin_7)
- net ROW2: now also J1.8 (Pin_8)
- net ROW3: now also J1.9 (Pin_9)
- net ROW4: now also J1.10 (Pin_10)
- net ROW5: now also J1.11 (Pin_11)
- net ROW6: now also J1.12 (Pin_12)
- net TO_Q1: now also J1.1 (Pin_1), Q1.3 (C)
- net TO_Q2: now also Q2.3 (C), J1.2 (Pin_2); no longer Q2.2 (C)
- net TO_Q3: now also Q3.3 (C), J1.3 (Pin_3); no longer Q3.2 (C)
- net TO_Q4: now also J1.4 (Pin_4), Q4.3 (C)
- net TO_Q5: now also Q5.3 (C), J1.5 (Pin_5); no longer Q5.2 (C)
- net TO_Q6: now also Q6.3 (C), J1.6 (Pin_6); no longer Q6.2 (C)
- net at R1.2: now also Q1.1 (B)
- net at R4.2: now also Q4.1 (B)
