File: hardware/top_board/top_board.kicad_sch (KiCad schematic)
At the start: 38 parts, among them J1 Conn_01x06, J2 Conn_01x06

Commit message: Recent changes
Parts:
- added J3: Conn_01x16_Pin, symbol Connector:Conn_01x16_Pin
Connections:
- net ROW1: now also J3.6 (Pin_6); no longer J1.1 (Pin_1)
- net ROW2: now also J3.5 (Pin_5); no longer J1.2 (Pin_2)
- net ROW3: now also J3.4 (Pin_4); no longer J1.3 (Pin_3)
- net ROW4: now also J3.3 (Pin_3); no longer J1.4 (Pin_4)
- net ROW5: now also J3.2 (Pin_2); no longer J1.5 (Pin_5)
- net ROW6: now also J3.1 (Pin_1); no longer J1.6 (Pin_6)
- net TO_Q1: now also J3.12 (Pin_12); no longer J2.1 (Pin_1)
- net TO_Q2: now also J3.11 (Pin_11); no longer J2.2 (Pin_2)
- net TO_Q3: now also J3.10 (Pin_10); no longer J2.3 (Pin_3)
- net TO_Q4: now also J3.9 (Pin_9); no longer J2.4 (Pin_4)
- net TO_Q5: now also J3.8 (Pin_8); no longer J2.5 (Pin_5)
- net TO_Q6: now also J3.7 (Pin_7); no longer J2.6 (Pin_6)
Changed lines of the file:
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@@
+		)
+	)
+	(label "ROW1"
+		(at 208.28 100.33 0)
+		(effects
+			(font
+				(size 1.27 1.27)
+			)
+			(justify left bottom)
 		)
 	)
@@
 		)
 	)
-	(label "ROW3"
-		(at 173.99 90.17 180)
+	(label "TO_Q1"
+		(at 208.28 115.57 0)
 		(effects
 			(font
 				(size 1.27 1.27)
 			)
-			(justify right bottom)
-		)
-	)
-	(label "TO_Q2"
-		(at 173.99 110.49 180)
+			(justify left bottom)
+		)
+	)
+	(label "ROW6"
+		(at 208.28 87.63 0)
 		(effects
 			(font
 				(size 1.27 1.27)
 			)
-			(justify right bottom)
-		)
-	)
-	(label "ROW6"
-		(at 173.99 97.79 180)
-		(effects
-			(font
-				(size 1.27 1.27)
-			)
-			(justify right bottom)
+			(justify left bottom)
 		)
 	)
@@
 		)
 	)
-	(label "ROW4"
-		(at 173.99 92.71 180)
+	(label "TO_Q4"
+		(at 208.28 107.95 0)
 		(effects
 			(font
 				(size 1.27 1.27)
 			)
-			(justify right bottom)
-		)
-	)
-	(label "ROW5"
-		(at 173.99 95.25 180)
+			(justify left bottom)
+		)
+	)
+	(label "ROW4"
+		(at 208.28 92.71 0)
 		(effects
 			(font
 				(size 1.27 1.27)
 			)
-			(justify right bottom)
+			(justify left bottom)
+		)
+	)
+	(label "ROW3"
+		(at 208.28 95.25 0)
+		(effects
+			(font
+				(size 1.27 1.27)
+			)
+			(justify left bottom)
 		)
 	)
@@
 		)
 	)
-	(label "TO_Q4"
-		(at 173.99 115.57 180)
-		(effects
-			(font
-				(size 1.27 1.27)
-			)
-			(justify right bottom)
-		)
-	)
 	(label "ROW3"
 		(at 147.32 100.33 0)
@@
 		)
 	)
-	(label "TO_Q5"
-		(at 173.99 118.11 180)
-		(effects
-			(font
-				(size 1.27 1.27)
-			)
-			(justify right bottom)
-		)
-	)
 	(label "TO_Q2"
 		(at 91.44 127 180)
@@
 		)
 	)
-	(label "ROW2"
-		(at 173.99 87.63 180)
+	(label "ROW5"
+		(at 208.28 90.17 0)
 		(effects
 			(font
 				(size 1.27 1.27)
 			)
-			(justify right bottom)
+			(justify left bottom)
 		)
 	)
 	(label "TO_Q3"
-		(at 173.99 113.03 180)
+		(at 208.28 110.49 0)
 		(effects
 			(font
 				(size 1.27 1.27)
 			)
-			(justify right bottom)
-		)
-	)
-	(label "TO_Q6"
-		(at 173.99 120.65 180)
+			(justify left bottom)
+		)
+	)
+	(label "TO_Q5"
+		(at 208.28 105.41 0)
 		(effects
 			(font
 				(size 1.27 1.27)
 			)
-			(justify right bottom)
+			(justify left bottom)
 		)
 	)
@@
 		)
 	)
+	(label "TO_Q2"
+		(at 208.28 113.03 0)
+		(effects
+			(font
+				(size 1.27 1.27)
+			)
+			(justify left bottom)
+		)
+	)
+	(label "TO_Q6"
+		(at 208.28 102.87 0)
+		(effects
+			(font
+				(size 1.27 1.27)
+			)
+			(justify left bottom)
+		)
+	)
 	(label "TO_Q6"
 		(at 134.62 127 180)
@@
 		)
 	)
-	(label "TO_Q1"
-		(at 173.99 107.95 180)
+	(label "ROW2"
+		(at 208.28 97.79 0)
 		(effects
 			(font
 				(size 1.27 1.27)
 			)
-			(justify right bottom)
+			(justify left bottom)
 		)
 	)
@@
 		)
 	)
-	(label "ROW1"
-		(at 173.99 85.09 180)
-		(effects
-			(font
-				(size 1.27 1.27)
-			)
-			(justify right bottom)
-		)
-	)
 	(symbol
 		(lib_id "Device:LED")
@@
 					(unit 1)
 				)
+			)
+		)
+	)
+	(symbol
+		(lib_id "Connector:Conn_01x16_Pin")
+		(at 203.2 105.41 0)
+		(unit 1)
+		(body_style 1)
+		(exclude_from_sim no)
+		(in_bom yes)
+		(on_board yes)
+		(in_pos_files yes)
+		(dnp no)
+		(fields_autoplaced yes)
+		(property "Reference" "J3"
+			(at 203.835 82.55 0)
+			(show_name no)
+			(do_not_autoplace no)
+			(effects
+				(font
+					(size 1.27 1.27)
+				)
+			)
+		)
+		(property "Value" "Conn_01x16_Pin"
+			(at 203.835 85.09 0)
+			(show_name no)
+			(do_not_autoplace no)
+			(effects
+				(font
+					(size 1.27 1.27)
+				)
+			)
+		)
+		(property "Footprint" ""
+			(at 203.2 105.41 0)
+			(hide yes)
+			(show_name no)
+			(do_not_autoplace no)
+			(effects
+				(font
+					(size 1.27 1.27)
+				)
+			)
+		)
+		(property "Datasheet" ""
+			(at 203.2 105.41 0)
+			(hide yes)
+			(show_name no)
+			(do_not_autoplace no)
+			(effects
+				(font
+					(size 1.27 1.27)
+				)
+			)
+		)
+		(property "Description" "Generic connector, single row, 01x16, script generated"
+			(at 203.2 105.41 0)
+			(hide yes)
+			(show_name no)
+			(do_not_autoplace no)
+			(effects
+				(font
+					(size 1.27 1.27)
+				)
+			)
+		)
+		(pin "15"
+		)
+		(pin "16"
+		)
+		(pin "2"
+		)
+		(pin "3"
+		)
+		(pin "13"
+		)
+		(pin "14"
+		)
+		(pin "6"
+		)
+		(pin "7"
+		)
+		(pin "8"
+		)
+		(pin "9"
+		)
+		(pin "1"
+		)
+		(pin "4"
+		)
+		(pin "5"
+		)
+		(pin "10"
+		)
+		(pin "11"
+		)
+		(pin "12"
+		)
+		(instances
+			(project "top_board"
+				(path "/d03ed85a-e44e-4f5a-82b4-54a22b909308"
+					(reference "J3")
+					(unit 1)
+				)
